File: 208_PROGRAM_CARD/208_PROGRAM_CARD.kicad_pcb (KiCad board)
At the start: 2 copper layers, 157.5 x 60.7 mm, 156 parts, among them J1 Pad, J10 Pad, J100 Pad, J101 Pad, J102 Pad, J103 Pad, J104 Pad, J105 Pad, J106 Pad, J107 Pad, J108 Pad, J109 Pad, J11 Pad, J110 Pad, J111 Pad, J112 Pad, J113 Pad, J114 02x28 Edge - 3.96mm, J115 Pad, J116 Pad, J117 Pad, J118 Pad, J119 Pad, J12 Pad, J120 Pad, J121 Pad, J122 Pad, J123 Pad, J124 Pad, J125 Pad, J126 Pad, J127 Pad, J128 Pad, J129 Pad, J13 Pad, J130 Pad, J131 Pad, J132 Pad, J133 Pad, J134 Pad, J135 Pad, J136 Pad, J137 Pad, J138 Pad, J139 Pad, J14 Pad, J140 Pad, J141 Pad, J142 Pad, J143 Pad, J144 Pad, J15 Pad, J16 Pad, J17 Pad, J18 Pad, J19 Pad, J2 Pad, J20 Pad, J21 Pad, J22 Pad, J23 Pad, J24 Pad, J25 Pad, J26 Pad, J27 Pad, J28 Pad, J29 Pad, J3 Pad, J30 Pad, J31 Pad, J32 Pad, J33 Pad, J34 Pad, J35 Pad, J354 Pad, J355 Pad, J356 Pad, J357 Pad, J358 Pad, J36 Pad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

Commit message: initial commit
Parts:
- removed J1, J10, J100, J109, J11, J113, J115, J116, J117, J118, J119, J12, J120, J121, J122, J123, J124, J125, J126, J127, J128, J129, J13, J130, J131, J132, J133, J134, J135, J136, J137, J138, J139, J14, J140, J141, J142, J143, J144, J15, J16, J17, J18, J19, J2, J20, J21, J22, J23, J24, J25, J26, J27, J28, J29, J3, J30, J31, J32, J33, J34, J35, J354, J355, J356, J357, J358, J36, J37, J38, J39, J4, J40, J41, J42, J43, J44, J45, J46, J47, J48, J49, J5, J50, J51, J52, J53, J54, J55, J56, J57, J58, J59, J6, J60, J61, J62, J63, J64, J65, J66, J67, J68, J69, J7, J70, J71, J72, J73, J74, J75, J76, J77, J78, J79, J8, J80, J81, J82, J83, J84, J85, J86, J87, J88, J89, J9, J90, J91, J92, J93, J94, J95, J96, J97, J98, J99: Pad, Buchla_Connectors:SolderWirePad_1x01_Drill0.9mm
- removed M1: Logo_150mil, Dunnington:Logo_150mil
- removed TR1, TR2, TR3, TR4, TR5: TRIM, Potentiometer_THT:Potentiometer_Bourns_3266W_Vertical
- added J145: Conn_01x08, Connector_PinSocket_2.54mm:PinSocket_1x10_P2.54mm_Vertical, F.Cu at (88.9, 106.7)
- added J167: Conn_01x10, Connector_PinSocket_2.54mm:PinSocket_1x10_P2.54mm_Vertical, F.Cu at (80.0, 106.7)
- added J168: Conn_01x10, Connector_PinSocket_2.54mm:PinSocket_1x10_P2.54mm_Vertical, F.Cu at (97.8, 106.7)
- added J169: Conn_01x10, Connector_PinSocket_2.54mm:PinSocket_1x10_P2.54mm_Vertical, F.Cu at (115.6, 106.7)
- added J170: Conn_01x10, Connector_PinSocket_2.54mm:PinSocket_1x10_P2.54mm_Vertical, F.Cu at (133.3, 106.7)
- added J171: Conn_01x10, Connector_PinSocket_2.54mm:PinSocket_1x10_P2.54mm_Vertical, F.Cu at (151.1, 106.7)
- added J172: Conn_01x10, Connector_PinSocket_2.54mm:PinSocket_1x10_P2.54mm_Vertical, F.Cu at (168.9, 106.7)
- added J173: Conn_01x10, Connector_PinSocket_2.54mm:PinSocket_1x10_P2.54mm_Vertical, F.Cu at (186.7, 106.7)
- added J174: Conn_01x10, Connector_PinSocket_2.54mm:PinSocket_1x10_P2.54mm_Vertical, F.Cu at (204.5, 106.7)
- J101, J106: value Pad -> Conn_01x40; footprint Buchla_Connectors:SolderWirePad_1x01_Drill0.9mm -> Connector_PinSocket_2.54mm:PinSocket_1x40_P2.54mm_Vertical
- J102, J103, J104, J105, J110, J111, J112: value Pad -> Conn_01x08; footprint Buchla_Connectors:SolderWirePad_1x01_Drill0.9mm -> Connector_PinSocket_2.54mm:PinSocket_1x10_P2.54mm_Vertical
- J107, J108: value Pad -> Conn_01x14; footprint Buchla_Connectors:SolderWirePad_1x01_Drill0.9mm -> Connector_PinSocket_2.54mm:PinSocket_1x14_P2.54mm_Vertical
- moved J101 109.4 mm to (78.7, 101.6), turned to 90 degrees
- moved S1 60.6 mm to (220.8, 50.9)
- moved J112 55.5 mm to (213.4, 106.7), turned to 0 degrees
- moved J107 51.4 mm to (181.6, 101.6), turned to 90 degrees
- moved J111 37.0 mm to (195.6, 106.7), turned to 0 degrees
- moved J102 35.9 mm to (106.7, 106.7)
- moved J106 33.8 mm to (78.7, 91.4), turned to 90 degrees
- moved J108 30.7 mm to (181.6, 91.4), turned to 90 degrees
- moved J105 27.0 mm to (160.0, 106.7)
- moved J103 20.5 mm to (124.5, 106.7)
- moved J110 18.5 mm to (177.8, 106.7), turned to 0 degrees
- moved J104 15.2 mm to (142.4, 106.7)
Connections:
- J101 pad 1: /SEQ_CV_OUT -> /SEQ_CV_SUM
- J102 pad 1: /CO_PITCH -> /MO_INDEX
- J103 pad 1: /CO_PITCH -> /MO_FREQ
- J105 pad 1: /CO_PITCH -> /TIMBRE_CV
- J106 pad 1: /EG_CV_OUT -> /SEQ_DRIVE_1
- J107 pad 1: /EG_CV_OUT -> /MO_RANGE
- J108 pad 1: /EG_CV_OUT -> /ENABLE_+13.5V
- J110 pad 1: /TIMBRE_CV -> /LPG_1_CV
- J111 pad 1: /TIMBRE_CV -> /LPG_2_CV
- J112 pad 1: /TIMBRE_CV -> /INV_FROM_PROG
- J114 pad 2b: Net-(J114-Pad2b) -> unconnected-(J114-Pin_2b-Pad2b)
- J114 pad 4a: Net-(J114-Pad4a) -> unconnected-(J114-Pin_4a-Pad4a)
- J114 pad 4b: Net-(J114-Pad4b) -> unconnected-(J114-Pin_4b-Pad4b)
- J114 pad 5b: Net-(J114-Pad5b) -> unconnected-(J114-Pin_5b-Pad5b)
- J114 pad 6a: Net-(J114-Pad6a) -> unconnected-(J114-Pin_6a-Pad6a)
- J114 pad 6b: Net-(J114-Pad6b) -> unconnected-(J114-Pin_6b-Pad6b)
Routing:
- net /SEQ_CV_OUT: track 22.8 -> 160.7 mm
- net /RANDOM_1_CV_OUT: track 53.9 -> 190.8 mm
- net /INV_TO_PROG: track 26.7 -> 163.6 mm
- net /KEY_CV_OUT: track 11.5 -> 145.8 mm
- net /EG_CV_OUT: track 23.4 -> 157.7 mm
- net /RANDOM_2_CV_OUT: track 18.2 -> 152.4 mm
- net /PRE_TO_PROG: track 28.1 -> 162.2 mm
- net /PULSER_OUT: track 17.4 -> 149.2 mm
- net /KEY_PRESSURE_OUT: track 12.2 -> 144.1 mm
- net /SEQ_CV_SUM: track 146.1 -> 98.9 mm, vias 1 -> 2
- net /SEQ_DRIVE_4: track 103.9 -> 139.7 mm, vias 1 -> 2
- net /SEQ_DRIVE_5: track 105.4 -> 137.9 mm, vias 1 -> 3
- net /SEQ_DRIVE_3: track 109.3 -> 135.4 mm, vias 1 -> 2
- net /SEQ_DRIVE_1: track 115.8 -> 138.5 mm, vias 1 -> 2
- net /SEQ_DRIVE_2: track 109.7 -> 131.7 mm
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Other:
- board size 157.5 x 60.7 mm -> 157.5 x 65.8 mm
- net class Default removed
- board text added: "1"
- board text added: "2"
- board text added: ">"
- board text added: "ATT"
- board text added: "CMPLX"
- board text added: "DEC"
- board text added: "DUR"
- board text added: "EG"
- board text added: "ENV D"
- board text added: "ENVELOPE"
- board text added: "FREQ."
- board text added: "GATE"
- board text added: "INDEX"
- board text added: "INV"
- board text added: "INVERT"
- board text added: "KEY"
- board text added: "LEVEL 1"
- board text added: "LEVEL 2"
- board text added: "MOD"
- board text added: "MOD."
- board text added: "MODE"
- board text added: "N"
- board text added: "OFFSET"
- board text added: "PERIOD"
- board text added: "PITCH"
- board text added: "PRESS"
- board text added: "PULSE SEQUENCE"
- board text added: "PULSER"
- board text added: "Para-Meta-Programmer"
- board text added: "RAND"
- board text added: "RAND1"
- board text added: "RAND2"
- board text added: "RNG"
- board text added: "S.R."
- board text added: "SEQ"
- board text added: "SEQUENCER"
- board text added: "TIMBRE"
- board text added: "VOLTAGE LEVELS"
- board text added: "W.S."

Commit message: update design
Parts:
- removed S1: ROWS, Dunnington:208_PROGRAM_CARD
Routing:
- net /TIMBRE_CV: track 28.9 -> 34.0 mm
- net /LPG_1_CV: track 32.3 -> 37.3 mm
Other:
- board text added: "ASSOCIATES"
- board text added: "Metaprogrammer"
- board text added: "V1"
- board text removed: "Para-Meta-Programmer"
