File: 208_PROGRAM_CARD/208_PROGRAM_CARD.kicad_sch (KiCad schematic)
At the start: 103 parts, among them J1 Pad, J10 Pad, J101 Conn_01x40, J102 Conn_01x08, J103 Conn_01x08, J104 Conn_01x08, J105 Conn_01x08, J106 Conn_01x40, J107 Conn_01x14, J108 Conn_01x14, J11 Pad, J110 Conn_01x08, J111 Conn_01x08, J112 Conn_01x08, J114 02x28 Edge - 3.96mm, J12 Pad, J13 Pad, J14 Pad, J145 Conn_01x08, J15 Pad, J16 Pad, J167 Conn_01x10, J168 Conn_01x10, J169 Conn_01x10, J17 Pad, J170 Conn_01x10, J171 Conn_01x10, J172 Conn_01x10, J173 Conn_01x10, J174 Conn_01x10, J18 Pad, J19 Pad, J2 Pad, J20 Pad, J21 Pad, J22 Pad, J23 Pad, J24 Pad, J25 Pad, J26 Pad, J27 Pad, J28 Pad, J29 Pad, J3 Pad, J30 Pad, J31 Pad, J32 Pad, J33 Pad, J34 Pad, J35 Pad, J354 Pad, J355 Pad, J356 Pad, J357 Pad, J358 Pad, J36 Pad, J37 Pad, J38 Pad, J39 Pad, J4 Pad, J40 Pad, J41 Pad, J42 Pad, J43 Pad, J44 Pad, J45 Pad, J46 Pad, J47 Pad, J48 Pad, J49 Pad, J5 Pad, J50 Pad, J51 Pad, J52 Pad, J53 Pad, J54 Pad, J55 Pad, J56 Pad, J57 Pad, J58 Pad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

Commit message: schematic items on canvas
Parts:
- removed M1: Logo_150mil, Dunnington:Logo_150mil, symbol 208_PROGRAM_CARD-rescue:Logo_150mil-Dunnington
Other:
- moved on the sheet: J101, J107, J167, J168, J169, J170, J171, J172, J173, J174

Commit message: update design
Parts:
- removed J1, J10, J11, J12, J13, J14, J15, J16, J17, J18, J19, J2, J20, J21, J22, J23, J24, J25, J26, J27, J28, J29, J3, J30, J31, J32, J33, J34, J35, J354, J355, J356, J357, J358, J36, J37, J38, J39, J4, J40, J41, J42, J43, J44, J45, J46, J47, J48, J49, J5, J50, J51, J52, J53, J54, J55, J56, J57, J58, J59, J6, J60, J61, J62, J63, J64, J65, J66, J67, J68, J69, J7, J70, J8, J9: Pad, Buchla_Connectors:SolderWirePad_1x01_Drill0.9mm, symbol 208_PROGRAM_CARD-rescue:Conn_01x01_Male-Connector
- removed TR1, TR2, TR3, TR4, TR5: TRIM, Potentiometer_THT:Potentiometer_Bourns_3266W_Vertical, symbol 208_PROGRAM_CARD-rescue:R_POT_TRIM_Small-Dunnington
- J114: value 02x28 Edge - 3.96mm -> 02x28 Edge - 3.96mm
Connections:
- net RANDOM_2_CV_OUT: no longer J114.16a (Pin_16a)
Other:
- note removed: "Bourns 3266W footprints for fine tune"
- note removed: "CMPLX"
- note removed: "ENVELOPE"
- note removed: "GATE"
- note removed: "MOD"
- note removed: "PULSER"
- note removed: "RANDOM"
- note removed: "SEQUENCER"
- moved on the sheet: J101, J102, J103, J104, J105, J107, J110, J111, J112, J114, J145, J167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

Commit message: updated part info
Parts:
- J101, J106: LCSC Part # (none) -> C358724
- J102, J103, J104, J105, J110, J111, J112, J145: value Conn_01x08 -> Conn_01x10; LCSC Part # (none) -> C350286
- J107, J108: LCSC Part # (none) -> C2979993
- J167, J168, J169, J170, J171, J172, J173, J174: LCSC Part # (none) -> C350286
Connections:
- net RANDOM_2_CV_OUT: now also J114.16a (Pin_16a)
Changed lines of the file:
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@@
 	(text "COLUMNS"
 		(exclude_from_sim no)
-		(at 195.326 188.976 0)
+		(at 179.07 192.278 0)
 		(effects
 			(font
-				(size 1.27 1.27)
+				(size 6.35 6.35)
 			)
 			(justify left bottom)
@@
 		(effects
 			(font
-				(size 1.27 1.27)
+				(size 6.35 6.35)
 			)
 			(justify left bottom)
@@
 		)
 	)
+	(label "RANDOM_2_CV_OUT"
+		(at 397.51 74.93 180)
+		(fields_autoplaced yes)
+		(effects
+			(font
+				(size 1.27 1.27)
+			)
+			(justify right bottom)
+		)
+	)
 	(label "KEY_P_OUT"
 		(at 214.63 62.23 90)
@@
 			)
 		)
+		(property "LCSC Part #" ""
+			(at 407.67 69.85 0)
+			(effects
+				(font
+					(size 1.27 1.27)
+				)
+				(hide yes)
+			)
+		)
 		(pin "10a"
 		)
@@
 			)
 		)
+		(property "LCSC Part #" ""
+			(at 464.82 68.58 0)
+			(effects
+				(font
+					(size 1.27 1.27)
+				)
+				(hide yes)
+			)
+		)
 		(pin "1"
 		)
@@
 			)
 		)
-		(property "Value" "Conn_01x08"
+		(property "Value" "Conn_01x10"
 			(at 200.66 199.39 90)
 			(effects
@@
 			)
 		)
+		(property "LCSC Part #" "C350286"
+			(at 199.39 203.2 0)
+			(effects
+				(font
+					(size 1.27 1.27)
+				)
+				(hide yes)
+			)
+		)
 		(pin "1"
 		)
@@
 			)
 		)
-		(property "Value" "Conn_01x08"
+		(property "Value" "Conn_01x10"
 			(at 200.66 260.35 90)
 			(effects
@@
 			)
 		)
+		(property "LCSC Part #" "C350286"
+			(at 199.39 264.16 0)
+			(effects
+				(font
+					(size 1.27 1.27)
+				)
+				(hide yes)
+			)
+		)
 		(pin "1"
 		)
@@
 			)
 		)
+		(property "LCSC Part #" "C350286"
+			(at 334.01 350.52 0)
+			(effects
+				(font
+					(size 1.27 1.27)
+				)
+				(hide yes)
+			)
+		)
 		(pin "1"
 		)
@@
 			)
 		)
+		(property "LCSC Part #" "C350286"
+			(at 270.51 350.52 0)
+			(effects
+				(font
+					(size 1.27 1.27)
+				)
+				(hide yes)
+			)
+		)
 		(pin "1"
 		)
@@
 			)
 		)
+		(property "LCSC Part #" "C358724"
+			(at 209.55 72.39 0)
+			(effects
+				(font
+					(size 1.27 1.27)
+				)
+				(hide yes)
+			)
+		)
 		(pin "1"
 		)
@@
 			)
 		)
+		(property "LCSC Part #" "C350286"
+			(at 207.01 350.52 0)
+			(effects
+				(font
+					(size 1.27 1.27)
+				)
+				(hide yes)
+			)
+		)
 		(pin "1"
 		)
@@
 			)
 		)
-		(property "Value" "Conn_01x08"
+		(property "Value" "Conn_01x10"
 			(at 200.66 278.13 90)
 			(effects
@@
 			)
 		)
+		(property "LCSC Part #" "C350286"
+			(at 199.39 281.94 0)
+			(effects
+				(font
+					(size 1.27 1.27)
+				)
+				(hide yes)
+			)
+		)
 		(pin "1"
 		)
@@
 			)
 		)
-		(property "Value" "Conn_01x08"
+		(property "Value" "Conn_01x10"
 			(at 200.66 311.15 90)
 			(effects
@@
 			)
 		)
+		(property "LCSC Part #" "C350286"
+			(at 199.39 314.96 0)
+			(effects
+				(font
+					(size 1.27 1.27)
+				)
+				(hide yes)
+			)
+		)
 		(pin "1"
 		)
@@
 			)
 		)
+		(property "LCSC Part #" "C2979993"
+			(at 290.83 82.55 0)
+			(effects
+				(font
+					(size 1.27 1.27)
+				)
+				(hide yes)
+			)
+		)
 		(pin "1"
 		)
@@
 			)
 		)
+		(property "LCSC Part #" "C358724"
+			(at 209.55 82.55 0)
+			(effects
+				(font
+					(size 1.27 1.27)
+				)
+				(hide yes)
+			)
+		)
 		(pin "1"
 		)
@@
 			)
 		)
+		(property "LCSC Part #" "C2979993"
+			(at 290.83 72.39 0)
+			(effects
+				(font
+					(size 1.27 1.27)
+				)
+				(hide yes)
+			)
+		)
 		(pin "1"
 		)
@@
 			)
 		)
+		(property "LCSC Part #" "C350286"
+			(at 229.87 350.52 0)
+			(effects
+				(font
+					(size 1.27 1.27)
+				)
+				(hide yes)
+			)
+		)
 		(pin "1"
 		)
@@
 			)
 		)
+		(property "LCSC Part #" "C350286"
+			(at 313.69 350.52 0)
+			(effects
+				(font
+					(size 1.27 1.27)
+				)
+				(hide yes)
+			)
+		)
 		(pin "1"
 		)
@@
 			)
 		)
-		(property "Value" "Conn_01x08"
+		(property "Value" "Conn_01x10"
 			(at 200.66 295.91 90)
 			(effects
@@
 			)
 		)
+		(property "LCSC Part #" "C350286"
+			(at 199.39 299.72 0)
+			(effects
+				(font
+					(size 1.27 1.27)
+				)
+				(hide yes)
+			)
+		)
 		(pin "1"
 		)
@@
 			)
 		)
+		(property "LCSC Part #" "C350286"
+			(at 250.19 350.52 0)
+			(effects
+				(font
+					(size 1.27 1.27)
+				)
+				(hide yes)
+			)
+		)
 		(pin "1"
 		)
@@
 			)
 		)
+		(property "LCSC Part #" "C350286"
+			(at 293.37 350.52 0)
+			(effects
+				(font
+					(size 1.27 1.27)
+				)
+				(hide yes)
+			)
+		)
 		(pin "1"
 		)
@@
 			)
 		)
+		(property "LCSC Part #" "C350286"
+			(at 184.15 350.52 0)
+			(effects
+				(font
+					(size 1.27 1.27)
+				)
+				(hide yes)
+			)
+		)
 		(pin "1"
 		)
@@
 			)
 		)
-		(property "Value" "Conn_01x08"
+		(property "Value" "Conn_01x10"
 			(at 200.66 245.11 90)
 			(effects
@@
 			)
 		)
+		(property "LCSC Part #" "C350286"
+			(at 199.39 248.92 0)
+			(effects
+				(font
+					(size 1.27 1.27)
+				)
+				(hide yes)
+			)
+		)
 		(pin "1"
 		)
@@
 			)
 		)
-		(property "Value" "Conn_01x08"
+		(property "Value" "Conn_01x10"
 			(at 200.66 214.63 90)
 			(effects
@@
 			)
 		)
+		(property "LCSC Part #" "C350286"
+			(at 199.39 218.44 0)
+			(effects
+				(font
+					(size 1.27 1.27)
+				)
+				(hide yes)
+			)
+		)
 		(pin "1"
 		)
@@
 			)
 		)
-		(property "Value" "Conn_01x08"
+		(property "Value" "Conn_01x10"
 			(at 200.66 229.87 90)
 			(effects
@@
 			(at 199.39 233.68 0)
 			(effects
+				(font
+					(size 1.27 1.27)
+				)
+				(hide yes)
+			)
+		)
+		(property "LCSC Part #" "C350286"
+			(at 199.39 233.68 0)
+			(effects
